File: PET-N/decoder.kicad_sch (KiCad schematic)
At the start: 5 parts, among them U1 74LS145

Commit message: PET-N r3
Parts:
- C1: LCSC (none) -> C14663
- C5, C6, C7: LCSC (none) -> C15008
- U1: LCSC (none) -> C2873068
Connections:
- net S1: no longer U1.15 (P0)
- new net S0: U1.15 (P0)
Changed lines of the file:
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@@
 		)
 	)
-	(global_label "S1"
+	(global_label "S0"
 		(shape input)
 		(at 69.85 104.775 180)
@@
 			)
 		)
+		(property "LCSC" "C14663"
+			(at 100.33 86.995 0)
+			(effects
+				(font
+					(size 1.27 1.27)
+				)
+				(hide yes)
+			)
+		)
 		(pin "2"
 		)
@@
 			)
 		)
+		(property "LCSC" "C2873068"
+			(at 88.5033 97.409 0)
+			(effects
+				(font
+					(size 1.27 1.27)
+				)
+				(hide yes)
+			)
+		)
 		(pin "4"
 		)
@@
 			)
 		)
+		(property "LCSC" "C15008"
+			(at 171.45 78.4859 0)
+			(effects
+				(font
+					(size 1.27 1.27)
+				)
+				(hide yes)
+			)
+		)
 		(pin "1"
 		)
@@
 			)
 		)
+		(property "LCSC" "C15008"
+			(at 158.75 78.4859 0)
+			(effects
+				(font
+					(size 1.27 1.27)
+				)
+				(hide yes)
+			)
+		)
 		(pin "1"
 		)
@@
 			(effects
 				(font
+					(size 1.27 1.27)
+				)
+				(hide yes)
+			)
+		)
+		(property "LCSC" "C15008"
+			(at 184.785 77.8509 0)
+			(effects
+				(font
