File: PET-N/i2c.kicad_sch (KiCad schematic)
At the start: 42 parts, among them J4 LINK3, Q1 BC859, Q2 BC859, Q25 BC859, Q26 BC859, Q27 BC859, Q28 BC859, Q3 BC859, Q4 BC859, Q5 BC859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

Commit message: PET-N r3
Parts:
- C3, C4: LCSC (none) -> C14663
- Q1, Q2, Q25, Q26, Q27, Q28, Q3, Q4, Q5, Q6, Q7, Q8: LCSC C3200239 -> C139450
- R1, R2, R21, R22, R23, R24, R25, R26, R27, R28, R29, R3, R30, R4, R43, R44, R45, R46, R47, R48, R49, R5, R6, R7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: LCSC (none) -> C25611
- U3, U4: LCSC (none) -> C2678764
