File: PET-N/petkn.kicad_pcb (KiCad board)
At the start: 2 copper layers, 386.1 x 102 mm, 260 parts, among them J1 Extended_PET_keyboard_connect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, J2 Conn_02x03_Odd_Even, J3 LINK3, J4 LINK3, J5 SPACE1, J6 SPACE2, J67 LINK67, Q1 BC859, Q10 BC808, Q11 BC848, Q12 BC808, Q13 BC848, Q14 BC808, Q15 BC848, Q16 BC808, Q17 BC848, Q18 BC808, Q19 BC848, Q2 BC859, Q20 BC808, Q21 BC848, Q22 BC808, Q23 BC848, Q24 BC808, Q25 BC859, Q26 BC859, Q27 BC859, Q28 BC859, Q29 BC848, Q3 BC859, Q30 BC848, Q31 BC848, Q32 BC848, Q4 BC859, Q5 BC859, Q6 BC859, Q7 BC859, Q8 BC859, Q9 BC848, SW1 KP "=", SW10 KP "0", SW11 R SHIFT, SW12 ">", SW14 "]", SW15 "@", SW16 L SHIFT, SW17 KP "+", SW18 KP "2", SW2 KP ".", SW20 "?", SW21 ",", SW22 "N", SW23 "V", SW24 "X", SW25 KP "3", SW26 KP "1", SW27 RETURN, SW28 ";", SW29 "M", SW3 NC ($10), SW30 "B", SW31 "C", SW32 "Z", SW320 S LOCK, SW33 KP "*", SW34 KP "5", SW36 ":", SW37 "K", SW38 "H", SW39 "F", SW4 STOP, SW40 "S", SW41 KP "6", SW42 KP "4", SW44 "L", SW45 "J", SW46 "G", SW47 "D", SW48 "A", SW49 KP "/"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

Commit message: new schematics version mainly complete
Parts:
- removed C1, C2, C3, C4: C, Capacitor_SMD:C_0603_1608Metric_Pad1.08x0.95mm_HandSolder
- removed C5, C6: 100u, Capacitor_SMD:C_1206_3216Metric_Pad1.33x1.80mm_HandSolder
- removed J2: Conn_02x03_Odd_Even, Connector_PinHeader_2.54mm:PinHeader_2x03_P2.54mm_Vertical
- removed J3: LINK3, Connector_PinHeader_2.54mm:PinHeader_2x02_P2.54mm_Vertical
- removed J5: SPACE1, Connector_PinHeader_2.54mm:PinHeader_2x02_P2.54mm_Vertical
- removed J6: SPACE2, Connector_PinHeader_2.54mm:PinHeader_2x02_P2.54mm_Vertical
- removed J67: LINK67, Connector_PinHeader_2.54mm:PinHeader_2x02_P2.54mm_Vertical
- removed Q1, Q2, Q25, Q26, Q27, Q28, Q3, Q4, Q5, Q6, Q7, Q8: BC859, Package_TO_SOT_SMD:SOT-23
- removed Q10, Q12, Q14, Q16, Q18, Q20, Q22, Q24: BC808, Package_TO_SOT_SMD:SOT-23
- removed Q11, Q13, Q15, Q17, Q19, Q21, Q23, Q29, Q30, Q31, Q32, Q9: BC848, Package_TO_SOT_SMD:SOT-23
- removed R1, R10, R11, R12, R126, R129, R13, R132, R133, R14, R15, R16, R17, R18, R19, R2, R20, R21, R22, R23, R24, R25, R26, R27, R28, R29, R3, R30, R31, R32, R33, R34, R35, R36, R37, R38, R39, R4, R40, R41, R42, R43, R44, R45, R46, R47, R48, R49, R5, R6, R7, R8, R9: 100k, Resistor_SMD:R_0805_2012Metric
- removed R100, R101, R102, R103, R104, R105, R106, R107, R108, R109, R110, R111, R112, R113, R114, R115, R116, R117, R118, R119, R120, R121, R122, R123, R124, R125, R50, R51, R52, R53, R54, R55, R56, R57, R58, R59, R60, R61, R62, R63, R64, R65, R66, R67, R68, R69, R70, R71, R72, R73, R74, R75, R76, R77, R78, R79, R80, R81, R82, R83, R84, R85, R86, R87, R88, R89, R90, R91, R92, R93, R94, R95, R96, R97, R98, R99: 390, Resistor_SMD:R_0805_2012Metric
- removed R127, R128, R130, R131: 10k, Resistor_SMD:R_0805_2012Metric
- removed U5: ~, petkn:THB Miniature Thumbstick THB001P
- added C10: 100n, Capacitor_SMD:C_0805_2012Metric_Pad1.18x1.45mm_HandSolder, B.Cu at (202.3, 136.7)
- added C11: 100n, Capacitor_SMD:C_0805_2012Metric_Pad1.18x1.45mm_HandSolder, B.Cu at (191.2, 136.8)
- added C12: 100n, Capacitor_SMD:C_0805_2012Metric_Pad1.18x1.45mm_HandSolder, B.Cu at (299.6, 92.9)
- added C13: 100n, Capacitor_SMD:C_0805_2012Metric_Pad1.18x1.45mm_HandSolder, B.Cu at (149.9, 137.0)
- added C14: 100n, Capacitor_SMD:C_0805_2012Metric_Pad1.18x1.45mm_HandSolder, B.Cu at (178.5, 136.9)
- added C15: 100u, Capacitor_SMD:C_1206_3216Metric_Pad1.33x1.80mm_HandSolder, B.Cu at (280.6, 140.7)
- added C16: 100u, Capacitor_SMD:C_1206_3216Metric_Pad1.33x1.80mm_HandSolder, B.Cu at (291.4, 58.5)
- added C17: 100n, Capacitor_SMD:C_0805_2012Metric_Pad1.18x1.45mm_HandSolder, B.Cu at (279.8, 131.0)
- added C18: 100u, Capacitor_SMD:C_1206_3216Metric_Pad1.33x1.80mm_HandSolder, B.Cu at (76.4, 131.7)
- added C8: 100n, Capacitor_SMD:C_0805_2012Metric_Pad1.18x1.45mm_HandSolder, B.Cu at (102.8, 136.4)
- added C9: 100n, Capacitor_SMD:C_0805_2012Metric_Pad1.18x1.45mm_HandSolder, B.Cu at (215.0, 136.7)
- added D1: 1N4448, Diode_SMD:D_0603_1608Metric, B.Cu at (257.9, 139.9)
- added J7: AVR-ISP-6, Connector_IDC:IDC-Header_2x03_P2.54mm_Vertical, F.Cu at (299.5, 63.2)
- added JP1: SolderJumper_2_Bridged, Jumper:SolderJumper-2_P1.3mm_Open_RoundedPad1.0x1.5mm, B.Cu at (80.0, 61.2)
- added JP10: SolderJumper_2_Bridged, Jumper:SolderJumper-2_P1.3mm_Bridged_RoundedPad1.0x1.5mm, F.Cu at (50.9, 131.9)
- added JP11: SolderJumper_2_Bridged, Jumper:SolderJumper-2_P1.3mm_Open_RoundedPad1.0x1.5mm, F.Cu at (50.9, 136.3)
- added JP2: SolderJumper_2_Bridged, Jumper:SolderJumper-2_P1.3mm_Open_RoundedPad1.0x1.5mm, B.Cu at (80.0, 57.7)
- added JP3: SolderJumper_2_Bridged, Jumper:SolderJumper-2_P1.3mm_Open_RoundedPad1.0x1.5mm, F.Cu at (46.8, 130.6)
- added JP4: SolderJumper_3_Bridged12, Jumper:SolderJumper-3_P1.3mm_Bridged12_RoundedPad1.0x1.5mm_NumberLabels, F.Cu at (248.1, 133.5)
- added JP6: SolderJumper_3_Bridged12, Jumper:SolderJumper-3_P1.3mm_Bridged12_RoundedPad1.0x1.5mm_NumberLabels, F.Cu at (61.7, 133.7)
- added JP7: SolderJumper_3_Bridged12, Jumper:SolderJumper-3_P1.3mm_Bridged12_RoundedPad1.0x1.5mm_NumberLabels, F.Cu at (65.8, 133.7)
- added JP8: SolderJumper_2_Bridged, Jumper:SolderJumper-2_P1.3mm_Open_RoundedPad1.0x1.5mm, F.Cu at (46.8, 136.2)
- added JP9: SolderJumper_2_Bridged, Jumper:SolderJumper-2_P1.3mm_Bridged_RoundedPad1.0x1.5mm, F.Cu at (46.8, 133.4)
- added U6: 74LS174, Package_SO:SO-16_3.9x9.9mm_P1.27mm, B.Cu at (197.2, 136.7)
- added U7: 74LS145, Package_SO:SO-16_3.9x9.9mm_P1.27mm, B.Cu at (220.1, 136.5)
- added U8: ATmega32A-A, Package_QFP:TQFP-44_10x10mm_P0.8mm, B.Cu at (309.6, 97.6)
- added Y1: ASE-xxxMHz, Oscillator:Oscillator_SMD_Abracon_ASE-4Pin_3.2x2.5mm, B.Cu at (255.9, 135.2)
- C7: value 100u -> 100n; footprint Capacitor_SMD:C_1206_3216Metric_Pad1.33x1.80mm_HandSolder -> Capacitor_SMD:C_0805_2012Metric_Pad1.18x1.45mm_HandSolder; moved to B.Cu
- J4: value LINK3 -> AVR-ISP-6; footprint Connector_PinHeader_2.54mm:PinHeader_2x02_P2.54mm_Vertical -> Connector_IDC:IDC-Header_2x03_P2.54mm_Vertical
- SW1, SW10, SW12, SW14, SW15, SW17, SW18, SW2, SW20, SW21, SW22, SW23, SW24, SW25, SW26, SW28, SW29, SW30, SW31, SW32, SW33, SW34, SW36, SW37, SW38, SW39, SW4, SW40, SW41, SW42, SW44, SW45, SW46, SW47, SW48, SW49, SW5, SW50, SW52, SW53, SW54, SW55, SW56, SW57, SW58, SW59, SW60, SW61, SW62, SW63, SW64, SW65, SW66, SW68, SW69, SW7, SW70, SW71, SW72, SW73, SW74, SW75, SW76, SW77, SW78, SW79, SW80, SW9: footprint petkn:SW_Cherry_MX_1.00u_PCB_with_LED -> petkn:SW_Cherry_MX_1.00u_PCB_with_RGB_LED
- SW11, SW16: footprint petkn:SW_Cherry_MX_2.00u_PCB_with_LED -> petkn:SW_Cherry_MX_2.00u_PCB_with_RGB_LED
- SW27, SW320, SW67, SW8: footprint petkn:SW_Cherry_MX_1.50u_PCB_with_LED -> petkn:SW_Cherry_MX_1.50u_PCB_with_RGB_LED
- SW3: footprint petkn:SW_Cherry_MX_1.25u_PCB_with_LED -> petkn:SW_Cherry_MX_1.25u_PCB_with_RGB_LED
- SW6: footprint petkn:SW_Cherry_MX_6.25u_PCB_with_LED -> petkn:SW_Cherry_MX_6.25u_PCB_with_RGB_LED
- U1: value 74LS145 -> LSF0204Q; footprint Package_DIP:DIP-16_W7.62mm -> Package_SO:TSSOP-14_4.4x5mm_P0.65mm; moved to B.Cu
- U2: value PCA9557PW -> ATmega32A-A; footprint Package_SO:TSSOP-16_4.4x5mm_P0.65mm -> Package_QFP:TQFP-44_10x10mm_P0.8mm; moved to B.Cu
- U3: value PCA9531PW -> 74HCT85; footprint Package_SO:TSSOP-16_4.4x5mm_P0.65mm -> Package_SO:SO-16_3.9x9.9mm_P1.27mm; moved to B.Cu
- U4: value PCA9531PW -> 74LS174; footprint Package_SO:TSSOP-16_4.4x5mm_P0.65mm -> Package_SO:SO-16_3.9x9.9mm_P1.27mm; moved to B.Cu
- moved U1 176.3 mm to (142.0, 137.1)
- moved U4 126.6 mm to (185.5, 136.7)
- moved U3 103.1 mm to (207.2, 136.7)
- moved C7 85.7 mm to (255.9, 131.2), turned to 0 degrees
- moved U2 58.9 mm to (268.5, 135.7), turned to -90 degrees
- moved J4 20.5 mm to (305.8, 75.6)
Connections:
- C7 pad 1: VCC -> V33
- J1 pad 11: R2 -> cR2
- J1 pad 12: R1 -> cR1
- J1 pad 28: SCL -> LVSCL
- J1 pad 29: SDA -> LVSDA
- J4 pad 1: R2 -> Net-(J4-MISO)
- J4 pad 2: /IRQ -> VCC
- J4 pad 3: R1 -> Net-(J4-SCK)
- J4 pad 4: /RES -> Net-(J4-MOSI)
- SW1 pad 3: Net-(SW1B-K) -> GND
- SW1 pad 4: HI3 -> L0
- SW10 pad 3: Net-(SW10B-K) -> GND
- SW10 pad 4: HI0 -> Net-(SW10B-DIN)
- SW11 pad 3: Net-(SW11B-K) -> GND
- SW11 pad 4: HI7 -> Net-(SW11B-DIN)
- SW12 pad 3: Net-(SW12B-K) -> GND
- SW12 pad 4: HI4 -> Net-(SW12B-DIN)
- SW14 pad 3: Net-(SW14B-K) -> GND
- SW14 pad 4: HI4 -> Net-(SW14B-DIN)
- SW15 pad 3: Net-(SW15B-K) -> GND
- SW15 pad 4: HI4 -> Net-(SW15B-DIN)
- SW16 pad 3: Net-(SW16B-K) -> GND
- SW16 pad 4: HI4 -> Net-(SW16B-DIN)
- SW17 pad 3: Net-(SW17B-K) -> GND
- SW17 pad 4: HI3 -> Net-(SW17B-DIN)
- SW18 pad 3: Net-(SW18B-K) -> GND
- SW18 pad 4: HI1 -> Net-(SW10B-DOUT)
- SW2 pad 3: Net-(R123-Pad1) -> GND
- SW2 pad 4: HI1 -> L1
- SW20 pad 3: Net-(SW20B-K) -> GND
- SW20 pad 4: HI6 -> Net-(SW12B-DOUT)
- SW21 pad 3: Net-(SW21B-K) -> GND
- SW21 pad 4: HI7 -> Net-(SW21B-DIN)
- SW22 pad 3: Net-(SW22B-K) -> GND
- SW22 pad 4: HI5 -> Net-(SW14B-DOUT)
- SW23 pad 3: Net-(SW23B-K) -> GND
- SW23 pad 4: HI3 -> Net-(SW15B-DOUT)
- SW24 pad 3: Net-(SW24B-K) -> GND
- SW24 pad 4: HI1 -> Net-(SW16B-DOUT)
- SW25 pad 3: Net-(SW25B-K) -> GND
- SW25 pad 4: HI2 -> Net-(SW17B-DOUT)
- SW26 pad 3: Net-(SW26B-K) -> GND
- SW26 pad 4: HI0 -> Net-(SW18B-DOUT)
- SW27 pad 3: Net-(SW27B-K) -> GND
- SW27 pad 4: unconnected-(SW27B-A-Pad4) -> Net-(SW11B-DOUT)
- SW28 pad 3: Net-(SW28B-K) -> GND
- SW28 pad 4: HI5 -> Net-(SW20B-DOUT)
- SW29 pad 3: Net-(SW29B-K) -> GND
- SW29 pad 4: HI6 -> Net-(SW21B-DOUT)
- SW3 pad 2: XR3 -> R10
- SW3 pad 3: Net-(R117-Pad1) -> GND
- SW3 pad 4: HI6 -> L2
- SW30 pad 3: Net-(SW30B-K) -> GND
- SW30 pad 4: HI4 -> Net-(SW22B-DOUT)
- SW31 pad 3: Net-(SW31B-K) -> GND
- SW31 pad 4: HI2 -> Net-(SW23B-DOUT)
- SW32 pad 3: Net-(SW32B-K) -> GND
- SW32 pad 4: HI0 -> Net-(SW24B-DOUT)
- SW320 pad 2: XR1 -> xR9
- SW320 pad 3: Net-(R86-Pad1) -> GND
- SW320 pad 4: HI4 -> Net-(SW320B-DIN)
- SW33 pad 3: Net-(SW33B-K) -> GND
- SW33 pad 4: HI3 -> Net-(SW25B-DOUT)
- SW34 pad 3: Net-(SW34B-K) -> GND
- SW34 pad 4: HI1 -> Net-(SW26B-DOUT)
- SW36 pad 3: Net-(SW36B-K) -> GND
- SW36 pad 4: HI1 -> Net-(SW28B-DOUT)
- SW37 pad 3: Net-(SW37B-K) -> GND
- SW37 pad 4: HI7 -> Net-(SW29B-DOUT)
- SW38 pad 3: Net-(SW38B-K) -> GND
- SW38 pad 4: HI5 -> Net-(SW30B-DOUT)
- SW39 pad 3: Net-(SW39B-K) -> GND
- SW39 pad 4: HI3 -> Net-(SW31B-DOUT)
- SW4 pad 3: Net-(SW4B-K) -> GND
- SW4 pad 4: unconnected-(SW4B-A-Pad4) -> L3
- SW40 pad 3: Net-(SW40B-K) -> GND
- SW40 pad 4: HI1 -> Net-(SW32B-DOUT)
- SW41 pad 3: Net-(SW41B-K) -> GND
- SW41 pad 4: HI2 -> Net-(SW33B-DOUT)
- SW42 pad 3: Net-(SW42B-K) -> GND
- SW42 pad 4: HI0 -> Net-(SW34B-DOUT)
- SW44 pad 3: Net-(SW44B-K) -> GND
- SW44 pad 4: HI0 -> Net-(SW36B-DOUT)
- SW45 pad 3: Net-(SW45B-K) -> GND
- SW45 pad 4: HI6 -> Net-(SW37B-DOUT)
- SW46 pad 3: Net-(SW46B-K) -> GND
- SW46 pad 4: HI4 -> Net-(SW38B-DOUT)
- SW47 pad 3: Net-(SW47B-K) -> GND
- SW47 pad 4: HI2 -> Net-(SW39B-DOUT)
- SW48 pad 3: Net-(SW48B-K) -> GND
- SW48 pad 4: HI0 -> Net-(SW40B-DOUT)
- SW49 pad 3: Net-(SW49B-K) -> GND
- SW49 pad 4: HI3 -> Net-(SW41B-DOUT)
- SW5 pad 3: Net-(SW5B-K) -> GND
- SW5 pad 4: HI3 -> L4
- SW50 pad 3: Net-(SW50B-K) -> GND
- SW50 pad 4: HI1 -> Net-(SW42B-DOUT)
- SW52 pad 3: Net-(SW52B-K) -> GND
- SW52 pad 4: HI1 -> Net-(SW44B-DOUT)
- SW53 pad 3: Net-(SW53B-K) -> GND
- SW53 pad 4: HI7 -> Net-(SW45B-DOUT)
- SW54 pad 3: Net-(SW54B-K) -> GND
- SW54 pad 4: HI5 -> Net-(SW46B-DOUT)
- SW55 pad 3: Net-(SW55B-K) -> GND
- SW55 pad 4: HI3 -> Net-(SW47B-DOUT)
- SW56 pad 3: Net-(SW56B-K) -> GND
- SW56 pad 4: HI1 -> Net-(SW48B-DOUT)
- SW57 pad 3: Net-(SW57B-K) -> GND
- SW57 pad 4: HI2 -> Net-(SW49B-DOUT)
- SW58 pad 3: Net-(SW58B-K) -> GND
- SW58 pad 4: HI0 -> Net-(SW50B-DOUT)
- SW59 pad 3: Net-(SW59B-K) -> GND
- SW59 pad 4: HI2 -> Net-(SW27B-DOUT)
- SW6 pad 3: Net-(SW6B-K) -> GND
- SW6 pad 4: HI5 -> L5
- SW60 pad 3: Net-(SW60B-K) -> GND
- SW60 pad 4: HI0 -> Net-(SW52B-DOUT)
- SW61 pad 3: Net-(SW61B-K) -> GND
- SW61 pad 4: HI6 -> Net-(SW53B-DOUT)
- SW62 pad 3: Net-(SW62B-K) -> GND
- SW62 pad 4: HI4 -> Net-(SW54B-DOUT)
- SW63 pad 3: Net-(SW63B-K) -> GND
- SW63 pad 4: HI2 -> Net-(SW55B-DOUT)
- SW64 pad 3: Net-(SW64B-K) -> GND
- SW64 pad 4: HI0 -> Net-(SW56B-DOUT)
- SW65 pad 3: Net-(SW65B-K) -> GND
- SW65 pad 4: HI3 -> Net-(SW57B-DOUT)
- SW66 pad 3: Net-(SW66B-K) -> GND
- SW66 pad 4: HI1 -> Net-(SW58B-DOUT)
- SW67 pad 3: Net-(R99-Pad1) -> GND
- SW67 pad 4: HI4 -> Net-(SW59B-DOUT)
- SW68 pad 3: Net-(SW68B-K) -> GND
- SW68 pad 4: HI1 -> Net-(SW60B-DOUT)
- SW69 pad 3: Net-(SW69B-K) -> GND
- SW69 pad 4: HI7 -> Net-(SW61B-DOUT)
- SW7 pad 3: Net-(SW7B-K) -> GND
- SW7 pad 4: HI3 -> L6
- SW70 pad 3: Net-(SW70B-K) -> GND
- SW70 pad 4: HI5 -> Net-(SW62B-DOUT)
- SW71 pad 3: Net-(SW71B-K) -> GND
- SW71 pad 4: HI3 -> Net-(SW63B-DOUT)
- SW72 pad 3: Net-(SW72B-K) -> GND
- SW72 pad 4: HI1 -> Net-(SW64B-DOUT)
- SW73 pad 3: Net-(SW73B-K) -> GND
- SW73 pad 4: HI2 -> Net-(SW65B-DOUT)
- SW74 pad 3: Net-(SW74B-K) -> GND
- SW74 pad 4: HI0 -> Net-(SW66B-DOUT)
- SW75 pad 3: Net-(SW75B-K) -> GND
- SW75 pad 4: HI2 -> Net-(SW67B-DOUT)
- SW76 pad 3: Net-(SW76B-K) -> GND
- SW76 pad 4: HI0 -> Net-(SW68B-DOUT)
- SW77 pad 3: Net-(SW77B-K) -> GND
- SW77 pad 4: HI6 -> Net-(SW69B-DOUT)
- SW78 pad 3: Net-(SW78B-K) -> GND
- SW78 pad 4: HI4 -> Net-(SW70B-DOUT)
- SW79 pad 3: Net-(SW79B-K) -> GND
- SW79 pad 4: HI2 -> Net-(SW71B-DOUT)
- SW8 pad 3: Net-(SW8B-K) -> GND
- SW8 pad 4: HI4 -> L7
- SW80 pad 3: Net-(SW80B-K) -> GND
- SW80 pad 4: HI0 -> Net-(SW72B-DOUT)
- SW9 pad 3: Net-(SW9B-K) -> GND
- SW9 pad 4: HI2 -> Net-(SW1B-DOUT)
- U1 pad 1: R1 -> VCC33
- U1 pad 10: R9 -> unconnected-(U1-B4-Pad10)
- U1 pad 11: R10 -> SDA
- U1 pad 12: S3 -> SCL
- U1 pad 13: S2 -> unconnected-(U1-B1-Pad13)
- U1 pad 14: S1 -> VCC
- U1 pad 2: R2 -> VCC33
- U1 pad 3: R3 -> LVSCL
- U1 pad 4: R4 -> LVSDA
- U1 pad 5: R5 -> VCC33
- U1 pad 6: R6 -> (no net)
- U1 pad 7: R7 -> GND
- U1 pad 8: GND -> VCC33
- U1 pad 9: R8 -> (no net)
- U2 pad 1: SCL -> Net-(J4-MOSI)
- U2 pad 10: ON3 -> Net-(U2-PD1)
- U2 pad 11: ON4 -> Net-(U2-PD2)
- U2 pad 12: ON5 -> Net-(D1-K)
- U2 pad 13: ON6 -> C4
- U2 pad 14: ON7 -> C5
- U2 pad 15: /IRQ -> C6
- U2 pad 16: VCC -> C7
- U2 pad 2: SDA -> Net-(J4-MISO)
- U2 pad 3: GND -> Net-(J4-SCK)
- U2 pad 4: GND -> Net-(J4-~{RST})
- U2 pad 5: GND -> VCC
- U2 pad 6: ON0 -> GND
- U2 pad 7: ON1 -> unconnected-(U2-XTAL2-Pad7)
- U2 pad 8: GND -> CLK16M
- U2 pad 9: ON2 -> Net-(U2-PD0)
- U3 pad 1: GND -> S3
- U3 pad 10: PWM5 -> Net-(U3-A0)
- U3 pad 11: PWM6 -> S1
- U3 pad 12: PWM7 -> Net-(U3-A1)
- U3 pad 13: /RES -> Net-(U3-A2)
- U3 pad 14: SCL -> S2
- U3 pad 15: SDA -> Net-(U3-A3)
- U3 pad 2: GND -> unconnected-(U3-Ia<b-Pad2)
- U3 pad 3: GND -> VCC
- U3 pad 4: PWM0 -> unconnected-(U3-Ia>b-Pad4)
- U3 pad 5: PWM1 -> unconnected-(U3-Oa>b-Pad5)
- U3 pad 6: PWM2 -> Net-(U2-PD2)
- U3 pad 7: PWM3 -> unconnected-(U3-Oa<b-Pad7)
- U3 pad 9: PWM4 -> S0
- U4 pad 10: unconnected-(U4-LED5-Pad10) -> Net-(U3-A2)
- U4 pad 11: unconnected-(U4-LED6-Pad11) -> Net-(U4-D3)
- U4 pad 12: unconnected-(U4-LED7-Pad12) -> Net-(U3-A1)
- U4 pad 13: /RES -> Net-(U4-D4)
- U4 pad 14: SCL -> Net-(U4-D5)
- U4 pad 15: SDA -> Net-(U3-A0)
- U4 pad 2: GND -> Net-(U4-D3)
- U4 pad 3: GND -> Net-(U4-D0)
- U4 pad 4: PWM8 -> Net-(U4-D1)
- U4 pad 5: PWM9 -> Net-(U4-D2)
- U4 pad 6: PWM10 -> Net-(U4-D2)
- U4 pad 7: PWM11 -> Net-(U3-A3)
- U4 pad 9: unconnected-(U4-LED4-Pad9) -> CLK16M
Routing:
- net VCC: track 1062.2 -> 0.00 mm, vias 54 -> 0
- net GND: track 964.2 -> 0.00 mm, vias 53 -> 0
- net R10: track 610.9 -> 0.00 mm, vias 10 -> 0
- net R9: track 600.6 -> 0.00 mm, vias 4 -> 0
- net HI2: track 551.1 -> 0.00 mm, vias 8 -> 0
- net HI3: track 494.2 -> 0.00 mm, vias 7 -> 0
- net HI0: track 488.4 -> 0.00 mm, vias 6 -> 0
- net R2: track 485.5 -> 0.00 mm, vias 7 -> 0
- net HI1: track 475.7 -> 0.00 mm, vias 3 -> 0
- net R8: track 462.7 -> 0.00 mm, vias 6 -> 0
- net C6: track 457.8 -> 0.00 mm, vias 4 -> 0
- net R4: track 455.1 -> 0.00 mm, vias 4 -> 0
- net HI4: track 449.4 -> 0.00 mm, vias 2 -> 0
- net R7: track 444.1 -> 0.00 mm, vias 4 -> 0
- net R5: track 420.0 -> 0.00 mm, vias 4 -> 0
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Other:
- board text added: "$0A"
- board text added: "$10"
- board text added: "ALT (SW13)"
- board text added: "ALT (SW51)"
- board text added: "SPACE"
- board text added: "SW3"
- board text added: "SW67"
- board text removed: "ALTERNATE"
- board text removed: "SW3=PRG"
- board text removed: "SW67=SPACE"
- board text removed: "SW67=TAB"

Commit message: first layout
Parts:
- moved JP4 184.2 mm to (64.0, 141.0)
- moved U4 42.6 mm to (142.9, 136.4)
- moved C14 42.6 mm to (136.0, 136.6)
- moved C13 31.9 mm to (118.1, 137.1)
- moved C7 28.7 mm to (284.6, 132.0), turned to 90 degrees
- moved Y1 23.9 mm to (279.6, 132.2)
- moved U1 16.8 mm to (125.2, 137.0)
- moved J7 15.7 mm to (306.6, 77.2), turned to 0 degrees
- moved J4 11.7 mm to (301.2, 64.8), turned to 90 degrees
- moved D1 11.1 mm to (259.2, 128.9)
- moved C11 9.75 mm to (181.5, 136.8)
- moved U6 8.89 mm to (188.3, 136.7)
- moved C17 5.87 mm to (279.9, 136.8)
- moved C10 4.61 mm to (197.7, 136.7)
- moved U3 2.30 mm to (204.9, 136.7)
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Routing:
- net VCC: track 0.00 -> 1611.3 mm, vias 0 -> 12
- net GND: track 0.00 -> 1428.4 mm, vias 0 -> 5
- net R4: track 0.00 -> 396.9 mm, vias 0 -> 1
- net R9: track 0.00 -> 395.0 mm, vias 0 -> 3
- net R5: track 0.00 -> 356.3 mm, vias 0 -> 4
- net C4: track 0.00 -> 342.1 mm, vias 0 -> 5
- net L7: track 0.00 -> 295.7 mm, vias 0 -> 4
- net R3: track 0.00 -> 251.3 mm
- net C1: track 0.00 -> 245.8 mm, vias 0 -> 4
- net Net-(SW320B-DIN): track 0.00 -> 241.4 mm, vias 0 -> 4
- net C7: track 0.00 -> 240.0 mm
- net Net-(SW15B-DIN): track 0.00 -> 230.3 mm, vias 0 -> 4
- net R8: track 0.00 -> 226.4 mm, vias 0 -> 2
- net C2: track 0.00 -> 215.7 mm, vias 0 -> 3
- net R6: track 0.00 -> 196.7 mm
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