File: PET-N/scanner.kicad_sch (KiCad schematic)
At the start: 15 parts, among them J4 AVR-ISP-6, U2 ATmega32A-A, U3 74HCT85, U4 74LS174, U6 74LS174, U7 74LS145, Y1 ASE-xxxMHz

Commit message: working on new layout
Parts:
- removed D1: 1N4448, Diode_SMD:D_SOD-323_HandSoldering, symbol PCM_Diode_AKL:1N4448
- added D78: 1N4448, Diode_SMD:D_SOD-323_HandSoldering, symbol PCM_Diode_AKL:1N4448
Connections:
- net at J4.5 (~{RST}): now also D78.1 (K); no longer U2.4 (~{RESET})
- net /RESOUT: now reaches U2.12 (PD3)
- new net /RESSCAN: D78.2 (A), U2.4 (~{RESET})
Changed lines of the file:
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@@
 	)
 	(junction
+		(at 208.28 159.385)
+		(diameter 0)
+		(color 0 0 0 0)
+	)
+	(junction
 		(at 247.65 36.195)
 		(diameter 0)
@@
 	(wire
 		(pts
-			(xy 144.78 81.915) (xy 148.59 81.915)
-		)
-		(stroke
-			(width 0)
-			(type default)
-		)
-	)
-	(wire
-		(pts
 			(xy 105.41 60.325) (xy 97.79 60.325)
 		)
@@
 	(wire
 		(pts
+			(xy 188.595 154.305) (xy 191.77 154.305)
+		)
+		(stroke
+			(width 0)
+			(type default)
+		)
+	)
+	(wire
+		(pts
 			(xy 66.04 131.445) (xy 63.5 131.445)
 		)
@@
 	(wire
 		(pts
+			(xy 208.28 159.385) (xy 208.28 161.925)
+		)
+		(stroke
+			(width 0)
+			(type default)
+		)
+	)
+	(wire
+		(pts
 			(xy 87.63 62.865) (xy 105.41 62.865)
 		)
@@
 	(wire
 		(pts
+			(xy 208.28 154.305) (xy 208.28 159.385)
+		)
+		(stroke
+			(width 0)
+			(type default)
+		)
+	)
+	(wire
+		(pts
 			(xy 264.16 137.795) (xy 269.875 137.795)
 		)
@@
 	(wire
 		(pts
+			(xy 188.595 147.955) (xy 188.595 154.305)
+		)
+		(stroke
+			(width 0)
+			(type default)
+		)
+	)
+	(wire
+		(pts
 			(xy 78.74 57.785) (xy 87.63 57.785)
 		)
@@
 	(wire
 		(pts
-			(xy 156.21 81.915) (xy 206.375 81.915)
+			(xy 161.925 83.185) (xy 206.375 83.185)
 		)
 		(stroke
@@
 	(wire
 		(pts
-			(xy 206.375 81.915) (xy 206.375 66.675)
+			(xy 206.375 83.185) (xy 206.375 66.675)
 		)
 		(stroke
@@
 	(wire
 		(pts
-			(xy 248.92 45.085) (xy 246.38 45.085)
+			(xy 184.15 147.955) (xy 188.595 147.955)
 		)
 		(stroke
@@
 	(wire
 		(pts
-			(xy 208.28 147.955) (xy 184.15 147.955)
+			(xy 248.92 45.085) (xy 246.38 45.085)
 		)
 		(stroke
@@
 	(wire
 		(pts
-			(xy 35.56 57.785) (xy 35.56 29.845)
+			(xy 199.39 154.305) (xy 208.28 154.305)
 		)
 		(stroke
@@
 	(wire
 		(pts
-			(xy 105.41 55.245) (xy 78.74 55.245)
+			(xy 35.56 57.785) (xy 35.56 29.845)
 		)
 		(stroke
@@
 	(wire
 		(pts
-			(xy 269.875 33.655) (xy 269.875 36.195)
+			(xy 105.41 55.245) (xy 78.74 55.245)
 		)
 		(stroke
@@
 	(wire
 		(pts
-			(xy 208.28 161.925) (xy 208.28 147.955)
+			(xy 269.875 33.655) (xy 269.875 36.195)
 		)
 		(stroke
@@
 	(wire
 		(pts
+			(xy 198.12 159.385) (xy 208.28 159.385)
+		)
+		(stroke
+			(width 0)
+			(type default)
+		)
+	)
+	(wire
+		(pts
 			(xy 66.04 80.645) (xy 66.04 78.105)
 		)
@@
 		)
 	)
+	(global_label "{slash}RESSCAN"
+		(shape input)
+		(at 198.12 159.385 180)
+		(fields_autoplaced yes)
+		(effects
+			(font
+				(size 1.27 1.27)
+			)
+			(justify right)
+		)
+		(property "Intersheetrefs" "${INTERSHEET_REFS}"
+			(at 185.9314 159.385 0)
+			(effects
+				(font
+					(size 1.27 1.27)
+				)
+				(justify right)
+				(hide yes)
+			)
+		)
+	)
 	(global_label "SDA"
 		(shape input)
@@
 		)
 	)
-	(global_label "{slash}RES"
-		(shape input)
-		(at 144.78 81.915 180)
+	(global_label "{slash}RESOUT"
+		(shape output)
+		(at 161.925 83.185 180)
 		(fields_autoplaced yes)
 		(effects
@@
 		)
 		(property "Intersheetrefs" "${INTERSHEET_REFS}"
-			(at 137.49 81.915 0)
+			(at 151.0064 83.185 0)
 			(effects
 				(font
@@
 	)
 	(symbol
+		(lib_id "PCM_Diode_AKL:1N4448")
+		(at 195.58 154.305 180)
+		(unit 1)
+		(exclude_from_sim no)
+		(in_bom yes)
+		(on_board yes)
+		(dnp no)
+		(fields_autoplaced yes)
+		(property "Reference" "D78"
+			(at 195.58 147.955 0)
+			(effects
+				(font
+					(size 1.27 1.27)
+				)
+			)
+		)
+		(property "Value" "1N4448"
+			(at 195.58 150.495 0)
+			(effects
+				(font
+					(size 1.27 1.27)
+				)
+			)
+		)
+		(property "Footprint" "Diode_SMD:D_SOD-323_HandSoldering"
+			(at 195.58 154.305 0)
+			(effects
+				(font
+					(size 1.27 1.27)
+				)
+				(hide yes)
+			)
+		)
+		(property "Datasheet" "https://datasheet.octopart.com/1N4448TR-ON-Semiconductor-datasheet-42765246.pdf"
+			(at 195.58 154.305 0)
+			(effects
+				(font
+					(size 1.27 1.27)
+				)
+				(hide yes)
+			)
+		)
+		(property "Description" "DO-35 Diode, Small Signal, Fast Switching, 75V, 150mA, 4ns, Alternate KiCad Library"
+			(at 195.58 154.305 0)
+			(effects
+				(font
+					(size 1.27 1.27)
+				)
+				(hide yes)
+			)
+		)
+		(pin "1"
+		)
+		(pin "2"
+		)
+		(instances
+			(project "petkn"
+				(path "/a0727808-af70-4056-b2ee-ab828c2acfbd/517ec251-9cce-431a-9802-232702808e0f"
+					(reference "D78")
+					(unit 1)
+				)
+			)
+		)
+	)
+	(symbol
 		(lib_id "power:VCC")
 		(at 133.35 140.335 0)
@@
 					(unit 1)
 				)
-			)
-		)
-	)
-	(symbol
-		(lib_id "PCM_Diode_AKL:1N4448")
-		(at 152.4 81.915 0)
-		(unit 1)
-		(exclude_from_sim no)
-		(in_bom yes)
-		(on_board yes)
-		(dnp no)
-		(fields_autoplaced yes)
-		(property "Reference" "D1"
-			(at 152.4 76.2 0)
-			(effects
-				(font
-					(size 1.27 1.27)
-				)
-			)
-		)
-		(property "Value" "1N4448"
-			(at 152.4 78.74 0)
-			(effects
-				(font
-					(size 1.27 1.27)
-				)
-			)
-		)
-		(property "Footprint" "Diode_SMD:D_SOD-323_HandSoldering"
-			(at 152.4 81.915 0)
-			(effects
-				(font
-					(size 1.27 1.27)
-				)
-				(hide yes)
-			)
-		)
-		(property "Datasheet" "https://datasheet.octopart.com/1N4448TR-ON-Semiconductor-datasheet-42765246.pdf"
-			(at 152.4 81.915 0)
-			(effects
-				(font
-					(size 1.27 1.27)
-				)
-				(hide yes)
-			)
-		)
-		(property "Description" "DO-35 Diode, Small Signal, Fast Switching, 75V, 150mA, 4ns, Alternate KiCad Library"
-			(at 152.4 81.915 0)
-			(effects
-				(font
-					(size 1.27 1.27)
-				)
-				(hide yes)
-			)
-		)
-		(pin "1"
-		)
-		(pin "2"
-		)
-		(instances
-			(project ""
-				(path "/a0727808-af70-4056-b2ee-ab828c2acfbd/517ec251-9cce-431a-9802-232702808e0f"
-					(reference "D1")
-					(unit 1)
-				)
