File: test/tidriver.kicad_sch (KiCad schematic)
At the start: 1 part, among them U6 TLC59108FPW

Commit message: work on 2nd update test
Parts:
- removed U6: TLC59108FPW, Package_SO:TSSOP-20_4.4x6.5mm_P0.65mm, symbol Driver_LED:TLC59108xPW
- added C10, C11, C12, C7, C8, C9: 100n, Capacitor_SMD:C_0805_2012Metric_Pad1.18x1.45mm_HandSolder, symbol Device:C
- added J1: AVR-ISP-6, Connector_IDC:IDC-Header_2x03_P2.54mm_Vertical, symbol Connector:AVR-ISP-6
- added U2: ATmega32A-A, Package_QFP:TQFP-44_10x10mm_P0.8mm, symbol MCU_Microchip_ATmega:ATmega32A-A
- added U3: 74HCT85, Package_SO:SO-16_3.9x9.9mm_P1.27mm, symbol 74xx:74HCT85
- added U4, U6: 74LS174, Package_SO:SO-16_3.9x9.9mm_P1.27mm, symbol 74xx:74LS174
- added U7: 74LS145, Package_SO:SO-16_3.9x9.9mm_P1.27mm, symbol 74xx:74LS145
- added Y1: ASE-xxxMHz, Oscillator:Oscillator_SMD_Abracon_ASE-4Pin_3.2x2.5mm, symbol Oscillator:ASE-xxxMHz
Connections:
- net GND: now also C10.2, C11.2, C12.2, C8.2, C9.2, J1.6 (GND), U2.18 (GND), U2.28 (GND), U2.39 (GND), U2.6 (GND), U3.8 (GND), U4.8 (GND), U6.8 (GND), U7.8 (GND), Y1.2 (GND)
- net SCL: now also U2.19 (PC0)
- net SDA: now also U2.20 (PC1)
- net VCC: now also C10.1, C11.1, C12.1, C8.1, C9.1, J1.2 (VCC), U2.17 (VCC), U2.27 (AVCC), U2.38 (VCC), U2.5 (VCC), U3.16 (VCC), U3.3 (Ia=b), U4.1 (~{Mr}), U4.16 (VCC), U6.1 (~{Mr}), U6.16 (VCC), U7.16 (VCC)
- new net: U4.4 (D1), U6.10 (Q3)
- new net: U4.13 (D4), U6.12 (Q4)
- new net: U6.13 (D4), U6.5 (Q1)
- new net: U6.14 (D5), U6.2 (Q0)
- new net: U4.14 (D5), U6.15 (Q5)
- new net: U4.3 (D0), U6.7 (Q2)
- new net: U3.13 (A2), U4.10 (Q3)
- new net: U4.11 (D3), U4.2 (Q0)
- new net: U3.12 (A1), U4.12 (Q4)
- new net: U3.10 (A0), U4.15 (Q5)
- new net: U4.5 (Q1), U4.6 (D2)
- new net: U3.15 (A3), U4.7 (Q2)
- new net: J1.1 (MISO), U2.2 (PB6)
- new net: J1.3 (SCK), U2.3 (PB7)
- new net: J1.4 (MOSI), U2.1 (PB5)
- new net: J1.5 (~{RST}), U2.4 (~{RESET})
- new net: U2.11 (PD2), U3.6 (Oa=b)
- new net: U2.22 (PC3), U7.12 (P3)
- new net: U2.21 (PC2), U7.13 (P2)
- new net: U2.10 (PD1), U7.14 (P1)
- new net: U2.9 (PD0), U7.15 (P0)
- new net: U2.12 (PD3), U2.44 (PB4)
- new net C1: U2.37 (PA0)
- new net C2: U2.36 (PA1)
- new net C3: U2.35 (PA2)
- new net C4: U2.34 (PA3)
- new net C5: U2.33 (PA4)
- new net C6: U2.32 (PA5)
- new net C7: U2.31 (PA6)
- new net C8: U2.30 (PA7)
- new net CLK16M: U2.8 (XTAL1), U4.9 (Cp), U6.9 (Cp), Y1.3 (OUT)
- new net Col0: U2.23 (PC4)
- new net Col1: U2.24 (PC5)
- new net Col2: U2.25 (PC6)
- new net Col3: U2.26 (PC7)
- new net Col4: U2.13 (PD4)
- new net Col5: U2.14 (PD5)
- new net Col6: U2.15 (PD6)
- new net Col7: U2.16 (PD7)
- new net Row0: U7.1 (Q0)
- new net Row1: U7.2 (Q1)
- new net Row2: U7.3 (Q2)
- new net Row3: U7.4 (Q3)
- new net Row4: U7.5 (Q4)
- new net Row5: U7.6 (Q5)
- new net Row6: U7.7 (Q6)
- new net Row7: U7.9 (Q7)
- new net Row8: U7.10 (Q8)
- new net Row9: U7.11 (Q9)
- new net S0: U2.40 (PB0), U3.9 (B0), U6.3 (D0)
- new net S1: U2.41 (PB1), U3.11 (B1), U6.4 (D1)
- new net S2: U2.42 (PB2), U3.14 (B2), U6.6 (D2)
- new net S3: U2.43 (PB3), U3.1 (B3), U6.11 (D3)
- new net V33: Y1.1 (EN), Y1.4 (Vdd)
Other:
- note added: "This AtMega translates keyboard maps - S0-S1 inputs are on port bits PB0-3, on a port not written to. Reason is they can be read and converted into a table index using ANDI #15 - PB4 could in theory be used to extend the keyboard mapping table, as fed from PD3. - PD2 is falling edge triggered interrupt, fed from the comparison between the S0-3 inputs and their delayed version. - U6 and U4 delay b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"
- note removed: "Device Address: 100XXXX = $40-$4F Selected: $40"

Commit message: work on 2nd update test
Connections:
- net GND: now also C7.2
- net V33: now also C7.1
Changed lines of the file:
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@@
 	)
 	(junction
+		(at 55.88 133.35)
+		(diameter 0)
+		(color 0 0 0 0)
+	)
+	(junction
 		(at 50.8 16.51)
 		(diameter 0)
@@
 	)
 	(junction
+		(at 45.72 115.57)
+		(diameter 0)
+		(color 0 0 0 0)
+	)
+	(junction
 		(at 179.07 35.56)
 		(diameter 0)
@@
 	(wire
 		(pts
+			(xy 35.56 133.35) (xy 55.88 133.35)
+		)
+		(stroke
+			(width 0)
+			(type default)
+		)
+	)
+	(wire
+		(pts
 			(xy 69.85 129.54) (xy 67.31 129.54)
 		)
@@
 	(wire
 		(pts
+			(xy 55.88 134.62) (xy 55.88 133.35)
+		)
+		(stroke
+			(width 0)
+			(type default)
+		)
+	)
+	(wire
+		(pts
 			(xy 274.32 24.13) (xy 274.32 21.59)
 		)
@@
 	(wire
 		(pts
+			(xy 55.88 133.35) (xy 55.88 132.08)
+		)
+		(stroke
+			(width 0)
+			(type default)
+		)
+	)
+	(wire
+		(pts
 			(xy 237.49 59.69) (xy 232.41 59.69)
 		)
@@
 	(wire
 		(pts
+			(xy 35.56 128.27) (xy 35.56 133.35)
+		)
+		(stroke
+			(width 0)
+			(type default)
+		)
+	)
+	(wire
+		(pts
 			(xy 232.41 128.27) (xy 237.49 128.27)
 		)
@@
 	(wire
 		(pts
+			(xy 35.56 120.65) (xy 35.56 115.57)
+		)
+		(stroke
+			(width 0)
+			(type default)
+		)
+	)
+	(wire
+		(pts
 			(xy 165.1 60.96) (xy 134.62 60.96)
 		)
@@
 		)
 	)
+	(wire
+		(pts
+			(xy 35.56 115.57) (xy 45.72 115.57)
+		)
+		(stroke
+			(width 0)
+			(type default)
+		)
+	)
 	(global_label "Col5"
 		(shape input)
@@
 	(symbol
 		(lib_id "power:GND")
-		(at 55.88 132.08 0)
+		(at 55.88 134.62 0)
 		(unit 1)
 		(exclude_from_sim no)
@@
 		(fields_autoplaced yes)
 		(property "Reference" "#PWR017"
-			(at 55.88 138.43 0)
+			(at 55.88 140.97 0)
 			(effects
 				(font
@@
 		)
 		(property "Value" "GND"
-			(at 55.88 137.16 0)
+			(at 55.88 139.7 0)
 			(effects
 				(font
@@
 		)
 		(property "Footprint" ""
-			(at 55.88 132.08 0)
+			(at 55.88 134.62 0)
 			(effects
 				(font
@@
 		)
 		(property "Datasheet" ""
-			(at 55.88 132.08 0)
+			(at 55.88 134.62 0)
 			(effects
 				(font
@@
 		)
 		(property "Description" "Power symbol creates a global label with name \"GND\" , ground"
-			(at 55.88 132.08 0)
+			(at 55.88 134.62 0)
 			(effects
 				(font

Commit message: production test pcb
Parts:
- C10, C11, C12, C7, C8, C9: LCSC (none) -> C14663
- J1: LCSC (none) -> C5372863
- U2: LCSC (none) -> C5659
- U3: LCSC (none) -> C5953
- U4, U6: LCSC (none) -> C6828
- U7: LCSC (none) -> C60829
- Y1: LCSC (none) -> C12668
Changed lines of the file:
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@@
+			)
+		)
+		(property "LCSC" "C6828"
+			(at 66.7319 76.2 0)
+			(effects
+				(font
+					(size 1.27 1.27)
+				)
+				(hide yes)
 			)
 		)
@@
 			)
 		)
+		(property "LCSC" "C14663"
+			(at 266.7 26.6699 0)
+			(effects
+				(font
+					(size 1.27 1.27)
+				)
+				(hide yes)
+			)
+		)
 		(pin "2"
 		)
@@
 			)
 		)
+		(property "LCSC" "C6828"
+			(at 118.8019 81.28 0)
+			(effects
+				(font
+					(size 1.27 1.27)
+				)
+				(hide yes)
+			)
+		)
 		(pin "12"
 		)
@@
 			)
 		)
+		(property "LCSC" "C5372863"
+			(at 168.91 140.9699 0)
+			(effects
+				(font
+					(size 1.27 1.27)
+				)
+				(hide yes)
+			)
+		)
 		(pin "1"
 		)
@@
 			)
 		)
+		(property "LCSC" "C14663"
+			(at 278.13 26.6699 0)
+			(effects
+				(font
+					(size 1.27 1.27)
+				)
+				(hide yes)
+			)
+		)
 		(pin "2"
 		)
@@
 			)
 		)
+		(property "LCSC" "C5953"
+			(at 174.6819 71.12 0)
+			(effects
+				(font
+					(size 1.27 1.27)
+				)
+				(hide yes)
+			)
+		)
 		(pin "16"
 		)
@@
 			)
 		)
+		(property "LCSC" "C14663"
+			(at 242.57 26.6699 0)
+			(effects
+				(font
+					(size 1.27 1.27)
+				)
+				(hide yes)
+			)
+		)
 		(pin "2"
 		)
@@
 			)
 		)
+		(property "LCSC" "C60829"
+			(at 135.1981 97.79 0)
+			(effects
+				(font
+					(size 1.27 1.27)
+				)
+				(hide yes)
+			)
+		)
 		(pin "16"
 		)
@@
 			)
 		)
+		(property "LCSC" "C14663"
+			(at 231.14 26.6699 0)
+			(effects
+				(font
+					(size 1.27 1.27)
+				)
+				(hide yes)
+			)
+		)
 		(pin "2"
 		)
@@
 			)
 		)
+		(property "LCSC" "C14663"
+			(at 255.27 26.6699 0)
+			(effects
+				(font
+					(size 1.27 1.27)
+				)
+				(hide yes)
+			)
+		)
 		(pin "2"
 		)
@@
 			)
 		)
+		(property "LCSC" "C14663"
+			(at 39.37 123.1899 0)
+			(effects
+				(font
+					(size 1.27 1.27)
+				)
+				(hide yes)
+			)
+		)
 		(pin "2"
 		)
@@
 			)
 		)
+		(property "LCSC" "C5659"
+			(at 250.5867 46.99 0)
+			(effects
+				(font
+					(size 1.27 1.27)
+				)
+				(hide yes)
+			)
+		)
 		(pin "5"
 		)
@@
 			(effects
 				(font
+					(size 1.27 1.27)
+				)
+				(hide yes)
+			)
+		)
+		(property "LCSC" "C12668"
+			(at 68.58 118.0398 0)
+			(effects
+				(font
